Commit message: ik issue solved, typo correction

File: franka_ros-develop/franka_description/robots/common/utils.xacro (robot description, xacro)
@@ -2,6 +2,6 @@
 <robot xmlns:xacro="http://www.ros.org/wiki/xacro">
   <!-- Load inertial properties. Property is implicitly passed to macros. -->
-  <xacro:property name="inertial_config" value="$(find franka_description)/robots/common/inertial.yaml"/>
-  <xacro:property name="inertial" value="${xacro.load_yaml(inertial_config)}"/>
+  <!--xacro:property name="inertial_config" value="$(find franka_description)/robots/common/inertial.yaml"/-->
+  <xacro:property name="inertial" value="${load_yaml('$(find franka_description)/robots/common/inertial.yaml')}"/>
   <!-- ============================================================== -->
   <!-- Macro to add an <inertial> tag based on yaml-load properties   -->
@@ -11,5 +11,5 @@
   <!-- ============================================================== -->
   <xacro:macro name="inertial_props" params="name inertial:=^">
-      <xacro:unless value="${name in inertial}">${xacro.warning('No inertia properties defined for: ' + name)}</xacro:unless>
+      <!--xacro:unless value="${name in inertial}">${xacro.warning('No inertia properties defined for: ' + name)}</xacro:unless-->
       <xacro:if value="${name in inertial}">
         <!-- Access inertia properties of link 'name' -->

File: franka_ros-develop/franka_description/robots/panda/panda.urdf.xacro (robot description, xacro)
@@ -19,5 +19,5 @@
   <xacro:arg name="rpy" default="0 0 0" />
   <xacro:franka_robot arm_id="$(arg arm_id)"
-                      joint_limits="${xacro.load_yaml('$(find franka_description)/robots/panda/joint_limits.yaml')}"
+                      joint_limits="${load_yaml('$(find franka_description)/robots/panda/joint_limits.yaml')}"
                       hand="$(arg hand)"
                       tcp_xyz="$(arg tcp_xyz)"
