Commit message: misc

File: custom_description/robots/custom_hand.xacro (robot description, xacro)
@@ -25,9 +25,9 @@
                 </geometry>
             </visual>
-            <!-- <collision>
+            <collision>
                 <geometry>
                     <mesh filename="package://custom_description/meshes/collision/camera.stl" />
                 </geometry>
-            </collision> -->
+            </collision>
         </link>
         <joint name="${arm_id}_hand_sc_joint" type="fixed">
@@ -54,9 +54,9 @@
                 </geometry>
             </visual>
-            <!-- <collision>
+            <collision>
                 <geometry>
                     <mesh filename="package://custom_description/meshes/collision/finger.stl"/>
                 </geometry>
-            </collision> -->
+            </collision>
         </link>
         <link name="${arm_id}_rightfinger">
@@ -67,10 +67,10 @@
                 </geometry>
             </visual>
-            <!-- <collision>
+            <collision>
                 <origin xyz="0 0 0" rpy="0 0 ${pi}"/>
                 <geometry>
                     <mesh filename="package://custom_description/meshes/collision/finger.stl"/>
                 </geometry>
-            </collision> -->
+            </collision>
         </link>
         <joint name="${arm_id}_finger_joint1" type="prismatic">
@@ -88,5 +88,5 @@
             <axis xyz="0 -1 0" />
             <limit effort="100" lower="0.0" upper="0.04" velocity="0.2" />
-            <!-- <mimic joint="${arm_id}_finger_joint1" /> -->
+            <mimic joint="${arm_id}_finger_joint1" />
             <dynamics damping="0.3" />
         </joint>

Commit message: description renew

File: custom_description/robots/custom_hand.xacro (robot description, xacro)
@@ -1,16 +1,11 @@
 <?xml version="1.0" encoding="utf-8"?>
 <robot xmlns:xacro="http://www.ros.org/wiki/xacro" name="hand">
+    <xacro:include filename="$(find custom_description)/robots/utils.xacro"/>
     <xacro:macro name="custom_hand" params="arm_id tcp_xyz tcp_rpy tcp2_xyz tcp2_rpy camera_xyz camera_rpy">
         <link name="${arm_id}_hand">
-            <visual>
-                <geometry>
-                    <mesh filename="package://custom_description/meshes/visual/hand.dae" />
-                </geometry>
-            </visual>
-            <collision>
-                <geometry>
-                    <mesh filename="package://custom_description/meshes/collision/hand.stl" />
-                </geometry>
-            </collision>
+            <xacro:visual name="hand" />
+            <xacro:visual name="camera" xyz="${camera_xyz}" rpy="${camera_rpy}" />
+            <xacro:collision name="hand"/>
+            <xacro:collision name="camera" xyz="${camera_xyz}" rpy="${camera_rpy}" />
         </link>
         <joint name="${arm_id}_hand_joint" type="fixed">
@@ -20,57 +15,29 @@
         </joint>
         <link name="${arm_id}_hand_sc">
-            <visual>
-                <geometry>
-                    <mesh filename="package://custom_description/meshes/visual/camera.dae" />
-                </geometry>
-            </visual>
             <collision>
                 <geometry>
-                    <mesh filename="package://custom_description/meshes/collision/camera.stl" />
+                    <sphere radius="0.14"/>
+                </geometry>
+            </collision>
+            <collision>
+                <origin xyz="0 0 0.14"/>
+                <geometry>
+                    <box size="0.04 0.14 0.14"/>
                 </geometry>
             </collision>
         </link>
         <joint name="${arm_id}_hand_sc_joint" type="fixed">
-            <origin xyz="${camera_xyz}" rpy="${camera_rpy}"/>
             <parent link="${arm_id}_hand" />
             <child link="${arm_id}_hand_sc" />
         </joint>
-        <link name="${arm_id}_hand_tcp" />
-        <link name="${arm_id}_hand_tcp2" />
-        <joint name="${arm_id}_hand_tcp_joint" type="fixed">
-            <origin xyz="${tcp_xyz}" rpy="${tcp_rpy}" />
-            <parent link="${arm_id}_hand" />
-            <child link="${arm_id}_hand_tcp" />
-        </joint>
-        <joint name="${arm_id}_hand_tcp2_joint" type="fixed">
-            <origin xyz="${tcp2_xyz}" rpy="${tcp2_rpy}" />
-            <parent link="${arm_id}_hand" />
-            <child link="${arm_id}_hand_tcp2" />
-        </joint>
+        <xacro:tcp name="tcp" xyz="${tcp_xyz}" rpy="${tcp_rpy}"/>
+        <xacro:tcp name="tcp2" xyz="${tcp2_xyz}" rpy="${tcp2_rpy}"/>
         <link name="${arm_id}_leftfinger">
-            <visual>
-                <geometry>
-                    <mesh filename="package://custom_description/meshes/visual/finger.dae" />
-                </geometry>
-            </visual>
-            <collision>
-                <geometry>
-                    <mesh filename="package://custom_description/meshes/collision/finger.stl"/>
-                </geometry>
-            </collision>
+            <xacro:visual name="finger"/>
+            <xacro:collision name="finger"/>
         </link>
         <link name="${arm_id}_rightfinger">
-            <visual>
-                <origin xyz="0 0 0" rpy="0 0 ${pi}" />
-                <geometry>
-                    <mesh filename="package://custom_description/meshes/visual/finger.dae" />
-                </geometry>
-            </visual>
-            <collision>
-                <origin xyz="0 0 0" rpy="0 0 ${pi}"/>
-                <geometry>
-                    <mesh filename="package://custom_description/meshes/collision/finger.stl"/>
-                </geometry>
-            </collision>
+            <xacro:visual name="finger" rpy="0 0 ${pi}"/>
+            <xacro:collision name="finger" rpy="0 0 ${pi}"/>
         </link>
         <joint name="${arm_id}_finger_joint1" type="prismatic">

Commit message: restore launch and advance robot description

File: custom_description/robots/custom_hand.xacro (robot description, xacro)
@@ -31,6 +31,6 @@
             <child link="${arm_id}_hand_sc" />
         </joint>
-        <xacro:tcp name="tcp" xyz="${tcp_xyz}" rpy="${tcp_rpy}"/>
-        <xacro:tcp name="tcp2" xyz="${tcp2_xyz}" rpy="${tcp2_rpy}"/>
+        <xacro:tcp name="grasp-tcp" parent="hand" xyz="${tcp_xyz}" rpy="${tcp_rpy}"/>
+        <xacro:tcp name="push-tcp" parent="hand" xyz="${tcp2_xyz}" rpy="${tcp2_rpy}"/>
         <link name="${arm_id}_leftfinger">
             <xacro:visual name="finger"/>

File: custom_description/robots/fr3.srdf.xacro (robot description, xacro)
@@ -3,11 +3,20 @@
     <xacro:include filename="$(find custom_description)/robots/utils.xacro" />
     <xacro:arg name="arm_id" default="panda" />
-    <group name="$(arg arm_id)_gripper">
-        <chain base_link="$(arg arm_id)_link0" tip_link="$(arg arm_id)_tcp" />
+    <group name="$(arg arm_id)_arm">
+        <chain base_link="$(arg arm_id)_link0" tip_link="$(arg arm_id)_link8" />
     </group>
-    <group name="$(arg arm_id)_pusher">
-        <chain base_link="$(arg arm_id)_link0" tip_link="$(arg arm_id)_tcp2" />
+    <group name="$(arg arm_id)_hand">
+        <link name="$(arg arm_id)_hand"/>
+        <link name="$(arg arm_id)_leftfinger"/>
+        <link name="$(arg arm_id)_rightfinger"/>
     </group>
-    <group_state name="ready" group="$(arg arm_id)_gripper">
+    <group name="$(arg arm_id)_manipulator">
+        <chain base_link="$(arg arm_id)_link0" tip_link="$(arg arm_id)_hand_push-tcp" />
+    </group>
+    <!-- <group name="$(arg arm_id)_body">
+        <group name="$(arg arm_id)_arm" />
+        <group name="$(arg arm_id)_hand" />
+    </group> -->
+    <group_state name="ready" group="$(arg arm_id)_manipulator">
         <joint name="$(arg arm_id)_joint1" value="0" />
         <joint name="$(arg arm_id)_joint2" value="${-pi/4}" />
@@ -17,6 +26,7 @@
         <joint name="$(arg arm_id)_joint6" value="${pi/2}" />
         <joint name="$(arg arm_id)_joint7" value="${pi/4}" />
+        <!-- <joint name="$(arg arm_id)_finger_joint1" value="0.04" /> -->
     </group_state>
-    <virtual_joint name="virtual_joint" type="fixed" parent_frame="world" child_link="$(arg arm_id)_link0" />
+    <!-- <virtual_joint name="$(arg arm_id)_virtual_joint" type="fixed" parent_frame="world" child_link="$(arg arm_id)_virtual_link" /> -->
     <xacro:configure_collisions link="link0" enabled="link5 link6 link7 hand" />
     <xacro:configure_collisions link="link1" enabled="link5 link6 link7 hand" />
@@ -24,7 +34,13 @@
     <xacro:configure_collisions link="link3" enabled="link7 hand" />
     <xacro:configure_collisions link="link4" enabled="hand"/>
-    <xacro:configure_collisions link="link5" />
-    <xacro:configure_collisions link="link6" />
+    <xacro:configure_collisions link="link5" enabled_fine="hand"/>
+    <xacro:configure_collisions link="link6" enabled_fine="hand"/>
     <xacro:configure_collisions link="link7" />
-    <xacro:configure_collisions link="hand" />
+    <xacro:configure_collisions link="hand" enabled_fine="link5 link6" />
+    <disable_collisions link1="$(arg arm_id)_leftfinger" link2="$(arg arm_id)_rightfinger" />
+    <disable_default_collisions link="$(arg arm_id)_base"/>
+    <enable_collisions link1="$(arg arm_id)_base" link2="$(arg arm_id)_hand_sc" />
+    <!-- <end_effector name="$(arg arm_id)_gripper" parent_link="$(arg arm_id)_tcp" group="$(arg arm_id)_hand" parent_group="$(arg arm_id)_manipulator"/> -->
+    <end_effector name="$(arg arm_id)_tcp2" parent_link="$(arg arm_id)_hand_push-tcp" group="$(arg arm_id)_hand" parent_group="$(arg arm_id)_manipulator"/>
+    <end_effector name="$(arg arm_id)_hand" parent_link="$(arg arm_id)_link8" group="$(arg arm_id)_hand" parent_group="$(arg arm_id)_arm" />
 </robot>

File: custom_description/robots/fr3.urdf.xacro (robot description, xacro)
@@ -1,27 +1,43 @@
 <?xml version='1.0' encoding='utf-8'?>
 <robot xmlns:xacro="http://www.ros.org/wiki/xacro" name="fr3">
-    <xacro:include filename="$(find franka_description)/robots/common/franka_robot.xacro"/>
+    <xacro:include filename="$(find franka_description)/robots/common/franka_arm.xacro"/>
     <xacro:include filename="$(find custom_description)/robots/custom_hand.xacro"/>
     <xacro:arg name="arm_id" default="panda"/>
-    <xacro:arg name="tcp_xyz" default="0 0 0.0934"/>
-    <xacro:arg name="tcp_rpy" default="0 0 0"/>
-    <xacro:arg name="tcp2_xyz" default="0 0 0.1974"/>
-    <xacro:arg name="tcp2_rpy" default="0 0 0"/>
-    <xacro:arg name="camera_xyz" default="0 0 0"/>
-    <xacro:arg name="camera_rpy" default="${pi} ${-pi/2} 0"/>
-    <xacro:franka_robot
+    <xacro:franka_arm
         arm_id="$(arg arm_id)"
+        safety_distance="0.03"
         joint_limits="${xacro.load_yaml('$(find franka_description)/robots/fr3/joint_limits.yaml')}"
-        hand="false"
         gazebo="false"
     />
     <xacro:custom_hand
         arm_id="$(arg arm_id)"
-        tcp_xyz="$(arg tcp_xyz)"
-        tcp_rpy="$(arg tcp_rpy)"
-        tcp2_xyz="$(arg tcp2_xyz)"
-        tcp2_rpy="$(arg tcp2_rpy)"
-        camera_xyz="$(arg camera_xyz)"
-        camera_rpy="$(arg camera_rpy)"
+        tcp_xyz="0 0 0.0934"
+        tcp_rpy="0 0 0"
+        tcp2_xyz="0 0 0.1974"
+        tcp2_rpy="0 0 0"
+        camera_xyz="0 0 0"
+        camera_rpy="${pi} ${-pi/2} 0"
     />
+    <link name="$(arg arm_id)_base">
+        <visual>
+            <origin xyz="-0.04 0 0.01"/>
+            <geometry>
+                <box size="0.25 0.2 0.02"/>
+            </geometry>
+            <material name="black">
+                <color rgba="0 0 0 1"/>
+            </material>
+        </visual>
+        <collision>
+            <origin xyz="-0.04 0 0.01"/>
+            <geometry>
+                <box size="0.25 0.2 0.02"/>
+            </geometry>
+        </collision>
+    </link>
+    <joint name="$(arg arm_id)_joint0" type="fixed">
+        <origin xyz="0 0 0.02"/>
+        <parent link="$(arg arm_id)_base"/>
+        <child link="$(arg arm_id)_link0"/>
+    </joint>
 </robot>

File: custom_description/robots/utils.xacro (robot description, xacro)
@@ -17,10 +17,10 @@
         </collision>
     </xacro:macro>
-    <xacro:macro name="tcp" params="name arm_id:=^ xyz rpy">
-        <link name="${arm_id}_${name}"/>
-        <joint name="${arm_id}_${name}_joint" type="fixed">
+    <xacro:macro name="tcp" params="name arm_id:=^ parent xyz rpy">
+        <link name="${arm_id}_${parent}_${name}"/>
+        <joint name="${arm_id}_${parent}_${name}_joint" type="fixed">
             <origin xyz="${xyz}" rpy="${rpy}"/>
-            <parent link="${arm_id}_hand"/>
-            <child link="${arm_id}_${name}"/>
+            <parent link="${arm_id}_${parent}"/>
+            <child link="${arm_id}_${parent}_${name}"/>
         </joint>
     </xacro:macro>
@@ -28,5 +28,5 @@
         <xacro:if value="${others}">
             <xacro:property name="other" value="${others.pop(0)}" />
-            <disable_collisions link1="${link}" link2="${other}" reason="Never" />
+            <disable_collisions link1="${link}" link2="${other}" />
             <xacro:disable_collisions_for />
         </xacro:if>
@@ -39,10 +39,10 @@
         </xacro:if>
     </xacro:macro>
-    <xacro:macro name="configure_collisions" params="link enabled:=''">
+    <xacro:macro name="configure_collisions" params="link enabled:='' enabled_fine:=''">
         <xacro:property name="env_fmt" value="$(arg arm_id)_{}" />
-        <xacro:disable_collisions_for link="${env_fmt.format(link)}" others="${[env_fmt.format('link%d'%i) for i in python.range(8)]+[env_fmt.format(j) for j in ['hand','leftfinger','rightfinger']]}" />
+        <xacro:disable_collisions_for link="${env_fmt.format(link)}" others="${python.list((python.set(env_fmt.format('link%d'%i) for i in python.range(8))|python.set(env_fmt.format(j) for j in ['hand','leftfinger','rightfinger']))-python.set(env_fmt.format(k) for k in enabled_fine.split()))}" />
         <xacro:property name="sc_fmt" value="$(arg arm_id)_{}_sc" />
         <disable_default_collisions link="${sc_fmt.format(link)}" />
-        <xacro:enable_collisions_for link="${sc_fmt.format(link)}" others="${[sc_fmt.format(j) for j in enabled.split()]}" />
+        <xacro:enable_collisions_for link="${sc_fmt.format(link)}" others="${python.list(python.set(sc_fmt.format(i) for i in enabled.split()))}" />
     </xacro:macro>
 </robot>

Commit message: LYS::Consolidation of Functions and Grasper & Pusher instance Initialized

File: custom_description/robots/custom_hand.xacro (robot description, xacro)
@@ -27,4 +27,5 @@
             </collision>
         </link>
+        <link/>
         <joint name="${arm_id}_hand_sc_joint" type="fixed">
             <parent link="${arm_id}_hand" />

File: custom_description/robots/fr3.urdf.xacro (robot description, xacro)
@@ -10,4 +10,5 @@
         gazebo="false"
     />
+    <xacro:if></xacro:if>
     <xacro:custom_hand
         arm_id="$(arg arm_id)"

Commit message: rollback and checked

File: custom_description/robots/custom_hand.xacro (robot description, xacro)
@@ -27,5 +27,4 @@
             </collision>
         </link>
-        <link/>
         <joint name="${arm_id}_hand_sc_joint" type="fixed">
             <parent link="${arm_id}_hand" />

File: custom_description/robots/fr3.srdf.xacro (robot description, xacro)
@@ -46,5 +46,5 @@
     <disable_default_collisions link="$(arg arm_id)_base"/>
     <enable_collisions link1="$(arg arm_id)_base" link2="$(arg arm_id)_hand_sc" />
-    <end_effector name="$(arg arm_id)_pusher" parent_link="$(arg arm_id)_hand_push-tcp" group="gripper" />
-    <end_effector name="$(arg arm_id)_grasper" parent_link="$(arg arm_id)_hand_grasp-tcp" group="gripper" />
+    <!-- <end_effector name="$(arg arm_id)_pusher" parent_link="$(arg arm_id)_hand_push-tcp" group="gripper" />
+    <end_effector name="$(arg arm_id)_grasper" parent_link="$(arg arm_id)_hand_grasp-tcp" group="gripper" /> -->
 </robot>

File: custom_description/robots/fr3.urdf.xacro (robot description, xacro)
@@ -10,5 +10,4 @@
         gazebo="false"
     />
-    <xacro:if></xacro:if>
     <xacro:custom_hand
         arm_id="$(arg arm_id)"
